File: Teensy 3.0 to Arduino R3/eagle/board.sch (EAGLE design)
At the start: 71 parts, among them IC1 78XX compatible, IC2 24AA256SN, IC3 24AA256SN, IC4 24AA256SN, IC5 24AA256SN, U1 MICROSD

Commit message: inital commit V4
Parts:
- removed JP14: (no value), SparkFun-Connectors:M02PTH
- added JP17, JP18: M10", SparkFun-Connectors:M10"
- added R25, R26, R27, R28, R29, R30, R31, R32, R33, R34, R35, R36, R37, R38, R39, R40, R41, R42: (no value), resistor:R-EU_R0805
- added SJ10, SJ11, SJ12, SJ13, SJ7, SJ8, SJ9: SOLDERJUMPERNO, SparkFun-Passives:SOLDERJUMPERNO
- added U$1: XBEE-1B2, SparkFun-RF:XBEE-1B2
- added U$3, U$4: M24, SparkFun-Connectors:M24
- C10: device rcl:CPOL-EUSANYO_SMD_E7 -> rcl:CPOL-EU085CS-1AR
- C3: device rcl:CPOL-EUA/3216-18W -> rcl:CPOL-EUCT3528
- JP12: value (none) -> PINHD-1X10; device adafruit:PINHD-1X13_BIG -> adafruit:PINHD-1X10
- JP13: device adafruit:PINHD-1X13_BIG -> adafruit:PINHD-1X8BIG
- JP16: device SparkFun-Connectors:M02PTH -> SparkFun-Connectors:M05PTH
- JP2: value M14 -> (none); device SparkFun-Connectors:M14 -> pinhead:PINHD-2X6
- JP3: value M10" -> M14; device SparkFun-Connectors:M10" -> SparkFun-Connectors:M14
- JP4: value M10" -> (none); device SparkFun-Connectors:M10" -> pinhead:PINHD-2X6
Connections:
- new net N$26: JP17.9, R26.2
- new net N$27: JP17.8, R27.2
- new net N$28: JP17.7, R28.2
- new net N$29: JP17.6, R29.2
- new net N$30: JP17.5, R30.2
- new net N$31: JP17.4, R31.2
- new net N$32: JP17.3, R32.2
- new net N$33: JP17.2, R33.2
- new net N$34: JP17.1, R34.2
- new net N$35: JP3.11, R35.2
- new net N$36: JP3.10, R36.2
- new net N$37: JP3.9, R37.2
- new net N$38: JP3.8, R38.2
- new net N$39: JP18.4, R39.2
- new net N$40: JP18.3, R40.2
- new net N$41: JP18.2, R41.2
- new net N$42: JP18.1, R42.2
- new net N$45: JP13.6, U$1.DIO12
- new net N$46: JP13.5, U$1.RESET
- new net N$47: JP13.4, U$1.RSSI
- new net N$48: JP13.3, U$1.DIO11
- new net N$49: JP13.2, U$1.RES@8
- new net N$50: JP13.1, U$1.DTR
- new net N$51: JP12.1, U$1.DIO0
- new net N$52: JP4.10, JP4.9, SJ10.1, SJ11.1, SJ12.1, SJ9.1
- new net N$53: JP4.11, JP4.12
- new net N$54: JP12.2, U$1.DIO1
- new net N$55: JP12.3, U$1.DIO2
- new net N$56: JP12.4, U$1.DIO3
- new net N$57: JP2.7, JP2.8
- new net N$58: JP2.10, JP2.9
- new net N$59: JP12.5, U$1.RTS
- new net N$60: JP12.6, U$1.DIO5
- new net N$61: JP12.7, U$1.RES@14
- new net N$62: JP12.8, U$1.DIO9
- new net N$63: JP12.9, U$1.CTS
- new net N$64: JP12.10, U$1.DIO4
- net 3.3V: now also JP16.4, JP2.3, JP2.4, JP2.5, JP2.6, JP3.12, SJ13.1, U$1.VDD, U$4.23; no longer JP12.1, JP13.13, JP14.1, JP2.12
- net 5V: now also SJ13.2; no longer JP14.2
- net A0: now also U$4.13
- net A1: now also U$4.14
- net A10: now also R42.1, U$4.2; no longer JP13.6, JP4.1
- net A11: now also R41.1, U$4.3; no longer JP13.7, JP4.2
- net A12: now also R40.1, U$4.4; no longer JP13.8, JP4.3
- net A13: now also R39.1, U$4.5; no longer JP13.9, JP4.4
- net A2: now also U$4.15
- net A3: now also U$4.16
- net A4: now also U$4.17
- net A5: now also U$4.18
- net A6: now also R38.1, U$4.19; no longer JP13.2, JP2.8
- net A7: now also R37.1, U$4.20; no longer JP13.3, JP2.9
- net A8: now also R36.1, U$4.21; no longer JP13.4, JP2.10
- net A9: now also R35.1, U$4.22; no longer JP13.5, JP2.11
- net AGND: now also JP3.13, U$4.24; no longer JP12.12, JP2.13
- net AREF: now also JP18.6, U$4.7; no longer JP4.6
- net D0: now also JP13.8, U$1.DOUT, U$3.24
- net D1: now also JP13.7, U$1.DIN, U$3.23
- net D10: now also SJ10.2, U$3.14
- net D11: now also JP2.11, JP2.12, JP4.5, JP4.6, U$3.13
- net D12: now also U$3.12
- net D13: now also JP4.7, JP4.8, U$4.12
- net D2: now also SJ11.2, SJ7.2, U$3.22
- net D24: now also R25.1, U$3.11; no longer JP12.2, JP3.10
- net D25: now also R26.1, U$3.10; no longer JP12.3, JP3.9
- net D26: now also R27.1, U$3.9; no longer JP12.4, JP3.8
- net D27: now also R28.1, U$3.8; no longer JP12.5, JP3.7
- net D28: now also R29.1, U$3.7; no longer JP12.6, JP3.6
- net D29: now also R30.1, U$3.6; no longer JP12.7, JP3.5
- net D3: now also SJ12.2, SJ8.2, U$3.21
- net D30: now also R31.1, U$3.5; no longer JP12.8, JP3.4
- net D31: now also R32.1, U$3.4; no longer JP12.9, JP3.3
- net D32: now also R33.1, U$3.3; no longer JP12.10, JP3.2
- net D33: now also R34.1, U$3.2; no longer JP12.11, JP3.1
- net D4: now also U$3.20
- net D5: now also U$3.19
- net D6: now also U$3.18
- net D7: now also U$3.17
- net D8: now also U$3.16
- net D9: now also SJ9.2, U$3.15
- net GND: now also JP16.3, JP18.9, JP2.1, JP2.2, JP4.1, JP4.2, JP4.3, JP4.4, U$1.GND, U$3.25, U$4.10; no longer JP12.13, JP13.1, JP4.9
- net N$10: now also JP3.7; no longer JP2.7
- net N$11: now also JP3.6; no longer JP2.6
- net N$12: now also JP3.5; no longer JP2.5
- net N$2: now also C10.+; no longer JP16.1
- net N$21: now also JP3.4; no longer JP2.4
- net N$22: now also JP3.3; no longer JP2.3
- net N$23: now also JP3.2; no longer JP2.2
- net N$24: now also JP3.1; no longer JP2.1
- net N$25: now also JP17.10, R25.2; no longer C10.+, JP16.2
- net PROG: now also JP16.2, JP18.5, U$4.6; no longer JP13.10, JP4.5
- net QW: now also SJ7.1, SJ8.1
- net RESET: now also JP16.1, JP18.7, U$4.8; no longer JP4.7
- net VBAT: now also JP16.5, JP18.10, U$4.11; no longer JP13.12, JP4.10
- net VIN: now also JP3.14, U$4.25; no longer JP2.14
- net VUSB: now also JP18.8, U$4.9; no longer JP13.11, JP4.8
Other:
- moved on the sheet: C10, C3, C4, F2, JP11, JP15, JP5, JP6, JP7, JP8, JP9, R3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

Commit message: -added RS485 transceiver
Parts:
- added C11: (no value), rcl:C-EUC0805K
- added IC6: LTC2862, maxim:MAX3468ESA
- added JP14: (no value), pinhead:PINHD-1X2
- added R43, R44, R45, R46, R47: (no value), resistor:R-EU_R0805
- added SJ14, SJ15, SJ16, SJ17: SOLDERJUMPERNO, SparkFun-Passives:SOLDERJUMPERNO
- added X2: (no value), con-wago-508:W237-03P
Connections:
- new net N$43: IC6.RE/, JP14.2, SJ16.2
- new net N$44: IC6.DE, JP14.1, SJ17.2
- new net N$65: IC6.B, R43.1, SJ14.1
- new net N$66: IC6.A, R44.1, SJ15.1
- new net RS485A: R44.2, R45.2, R47.1, SJ15.2, X2-2.KL
- new net RS485B: R43.2, R46.1, R47.2, SJ14.2, X2-3.KL
- net 3.3V: now also C11.1, IC6.VCC, R46.2
- net D4: now also SJ16.1, SJ17.1
- net D7: now also IC6.RO
- net D8: now also IC6.DI
- net GND: now also C11.2, IC6.GND, R45.1, X2-1.KL
Other:
- note added: "RS485"
- note added: "RS485A"
- note added: "RS485B"
- note added: "Serial1"
- note added: "Serial3"
- note added: "WIZ820io"
- note added: "XBee"
- note removed: "Additional header"
- moved on the sheet: JP11, JP12, JP13, JP16, JP2, JP4, JP5, JP6, JP7, JP8, JP9, R3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

Commit message: added Li Battery Charger, variometer, temperature sensor
Parts:
- removed JP10: (no value), SparkFun-Connectors:M03PTH
- removed JP12: PINHD-1X10, adafruit:PINHD-1X10
- removed JP13: (no value), adafruit:PINHD-1X8BIG
- added C12, C13, C16, C17: CAPACITOR-0805, thewknd:CAPACITOR-0805
- added CN3: (no value), adafruit:JST_2PIN-THM-RA
- added IC7: TMP102, thewknd:TMP102
- added IC8: MS5803-01BA, thewknd:MS5803-01BA
- added IC9: MCP73871, thewknd:MCP73871
- added P1, P10, P11, P12, P13, P2, P3, P4, P5, P6, P7, P8, P9: LED, thewknd:LED
- added Q1, Q2, Q3, Q4, Q5, Q6, Q7: 2N7002, adafruit:MOSFET-NREFLOW
- added R48, R49, R50, R51, R52, R53, R54, R55, R56, R57, R58, R59, R60, R61, R62, R63, R64, R65, R66: RESISTOR, thewknd:RESISTOR
- added SJ18, SJ19, SJ20, SJ25, SJ26, SJ27, SJ28, SJ29, SJ30: SOLDERJUMPERNO, SparkFun-Passives:SOLDERJUMPERNO
- added SJ21, SJ22, SJ23, SJ24: (no value), SparkFun-Passives:SOLDERJUMPER_2WAYT
- added X3, X4, X5: HEADER-2X2, thewknd:HEADER-2X2
- added X6: HEADER-2X10SLK, thewknd:HEADER-2X10SLK
- C1, C2: value (none) -> CAPACITOR_POL-3216-POL; device resistor:CPOL-EUCT3216 -> thewknd:CAPACITOR_POL-3216-POL
- C11, C4, C5, C6, C7, C8: value (none) -> CAPACITOR-0805; device rcl:C-EUC0805K -> thewknd:CAPACITOR-0805
- C3: value (none) -> CAPACITOR_POL-3216-POL; device rcl:CPOL-EUCT3528 -> thewknd:CAPACITOR_POL-3216-POL
- F1, F2: value (none) -> FUSE1812; device adafruit:PTCFUSE-1812 -> thewknd:FUSE1812
- IC2, IC3, IC4, IC5: value 24AA256SN -> 24AA1025SM; device microchip:24AA256SN -> thewknd:EEPROM24AAXXXSM
- R1, R10, R11, R12, R13, R14, R15, R16, R17, R18, R19, R2, R20, R21, R22, R23, R24, R25, R26, R27, R28, R29, R3, R30, R31, R32, R33, R34, R35, R36, R37, R38, R39, R40, R41, R42, R43, R44, R45, R46, R47, R5, R6, R7, R8, R9: value (none) -> RESISTOR; device resistor:R-EU_R0805 -> thewknd:RESISTOR
- R4: value (none) -> R4; device resistor:R-EU_R0805 -> thewknd:RESISTOR
Connections:
- new net /PG: IC9./PG, P12.C
- new net BAT_CHARGER: C17.1, IC9.IN1, X4.1, X4.3
- new net CE: IC9.CE, SJ24.2
- new net DIO0: U$1.DIO0, X6.2
- new net DIO1: U$1.DIO1, X6.4
- new net DIO11: U$1.DIO11, X6.13
- new net DIO12: U$1.DIO12, X6.7
- new net DIO2: U$1.DIO2, X6.6
- new net DIO3: U$1.DIO3, X6.8
- new net DIO4: U$1.DIO4, X6.20
- new net DIO5: U$1.DIO5, X6.12
- new net DIO9: U$1.DIO9, X6.16
- new net N$100: C16.1, CN3.2, IC9.VBAT1
- new net N$103: R43.1, R44.1, R49.1
- new net N$104: IC9.THERM, R43.2
- new net N$105: IC9.PROG3, R50.1
- new net N$106: IC9.PROG1, R51.1
- new net N$107: IC9.VPCC, R52.1, R53.2
- new net N$109: C2.+, C9.+, D2.A, IC1.VO, SJ2.1, X5.2, X5.4
- new net N$110: X4.2, X5.1
- new net N$111: P12.A, R54.2
- new net N$112: P11.A, R55.2
- new net N$113: P10.A, R56.2
- new net N$67: Q1.G, SJ20.1
- new net N$68: Q2.G, SJ25.2
- new net N$69: Q5.G, SJ28.1
- new net N$70: Q3.G, SJ26.1
- new net N$71: Q4.G, SJ27.2
- new net N$72: P8.A, R65.1
- new net N$73: P9.A, R64.1
- new net N$74: P13.A, R66.1
- new net PROG2: IC9.PROG2, SJ22.2
- new net SEL: IC9.SEL, SJ21.2
- new net STAT1: IC9.STAT1/LBO, P10.C
- new net STAT2: IC9.STAT2, P11.C
- new net TE: IC9./TE, SJ23.2
- new net VCC: C12.1, IC7.VCC, R48.1
- new net XBEE_CTS: U$1.CTS, X6.18
- new net XBEE_DIN: SJ30.2, U$1.DIN, X6.5
- new net XBEE_DOUT: SJ29.2, U$1.DOUT, X6.3
- new net XBEE_DTR: U$1.DTR, X6.17
- new net XBEE_RES1: U$1.RES@8, X6.15
- new net XBEE_RSSI: R65.2, U$1.RSSI, X6.11
- new net XBEE_RST: U$1.RESET, X6.9
- new net XBEE_RTS: R64.2, U$1.RTS, X6.10
- new net XBEE_VREF: U$1.RES@14, X6.14
- net 3.3V: now also C13.1, IC8.CSB, IC8.PS, IC8.VDD, R48.2, R53.1, R54.1, R55.1, R56.1, R57.2, R58.2, R59.2, R60.2, R61.2, R62.2, R63.2, R66.2, SJ21.3, SJ22.3, SJ23.3, SJ24.3, X5.3, X6.1; no longer C2.+, C9.+, D2.A, IC1.VO, SJ2.1
- net A4: now also IC7.SDA, IC8.SDI/SDA
- net A5: now also IC7.SCL, IC8.SCLK
- net A6: now also SJ12.2, SJ8.2
- net A7: now also SJ11.2, SJ7.2
- net AREF: now also SJ15.2; no longer JP5.8
- net D0: now also SJ25.1, SJ29.1; no longer JP13.8, U$1.DOUT
- net D1: now also SJ20.2, SJ30.1; no longer JP13.7, U$1.DIN
- net D10: now also SJ18.1
- net D11: no longer JP2.11, JP2.12
- net D12: now also JP2.11, JP2.12
- net D2: no longer SJ11.2, SJ7.2
- net D3: no longer SJ12.2, SJ8.2
- net D4: now also SJ3.2; no longer SJ16.1, SJ17.1
- net D5: now also SJ4.2
- net D6: now also SJ16.1, SJ17.1
- net D7: now also SJ26.2; no longer SJ3.2
- net D8: now also SJ27.1; no longer SJ4.2
- net D9: now also SJ19.1
- net EXT_POWER: now also F2.P$1; no longer F1.1
- net GND: now also C12.2, C13.2, C16.2, C17.2, CN3.1, IC7.ADD0, IC7.GND, IC8.GND, IC9.GND1, P13.C, P8.C, P9.C, Q1.S, Q2.S, Q3.S, Q4.S, Q5.S, Q6.S, Q7.S, R44.2, R49.2, R50.2, R51.2, R52.2, SJ21.1, SJ22.1, SJ23.1, SJ24.1, X6.19
- net N$1: now also F2.P$2, X3.2, X3.4; no longer F1.2, JP10.2
- net N$2: now also F1.P$2, SJ14.1; no longer C10.+, F2.2
- net N$3: now also X3.1; no longer JP10.1
- net N$44: now also SJ28.2
- net N$45: now also P5.C, Q5.D; no longer JP13.6, U$1.DIO12
- net N$46: now also P5.A, R57.1; no longer JP13.5, U$1.RESET
- net N$47: now also P4.A, R59.1; no longer JP13.4, U$1.RSSI
- net N$48: now also P3.A, R58.1; no longer JP13.3, U$1.DIO11
- net N$49: now also P3.C, Q4.D; no longer JP13.2, U$1.RES@8
- net N$50: now also P4.C, Q3.D; no longer JP13.1, U$1.DTR
- net N$51: now also P1.A, R61.1; no longer JP12.1, U$1.DIO0
- net N$54: now also P2.A, R60.1; no longer JP12.2, U$1.DIO1
- net N$55: now also P1.C, Q2.D; no longer JP12.3, U$1.DIO2
- net N$56: now also P2.C, Q1.D; no longer JP12.4, U$1.DIO3
- net N$59: now also P7.A, R63.1; no longer JP12.5, U$1.RTS
- net N$60: now also P6.A, R62.1; no longer JP12.6, U$1.DIO5
- net N$61: now also P6.C, Q7.D; no longer JP12.7, U$1.RES@14
- net N$62: now also P7.C, Q6.D; no longer JP12.8, U$1.DIO9
- net N$63: now also JP5.8, SJ15.1; no longer JP12.9, U$1.CTS
- net N$64: now also Q7.G, SJ18.2; no longer JP12.10, U$1.DIO4
- net N$65: now also C10.+, SJ14.2; no longer IC6.B, R43.1, SJ14.1
- net N$66: now also Q6.G, SJ19.2; no longer IC6.A, R44.1, SJ15.1
- net RS485A: now also IC6.A; no longer R44.2, SJ15.2
- net RS485B: now also IC6.B; no longer R43.2, SJ14.2
- net VIN: now also IC9.OUT1, X3.3; no longer JP10.3
- net VUSB: now also F1.P$1, X4.4; no longer F2.1
Other:
- note added: "I2C address: 1001000"
- note added: "I2C address: 1110110"
- note added: "MCP73871"
- note added: "MS5803-01BA"
- note added: "POWER LED"
- note added: "Serial1 LED"
- note added: "Serial2 LED"
- note added: "Serial3 LED"
- note added: "TMP102"
- note removed: "REG."
- moved on the sheet: BAT1, C10, C11, C5, C6, C7, C8, D1, IC6, JP11, JP14, JP15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
