File: EAGLEPCB/board.brd (EAGLE design)
At the start: 100 x 64.1 mm, 125 parts, among them J1 JACK-DC-3P-3410020P1, J2 CONNECTOR-HEADER-10P-3460510P1, J3 CONNECTOR-HEADER-10P-3460510P1, J4 MICRO-SDCARD-CONNECTOR-330006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, J5 JST-2P-SMD-PW, J6 MICRO-USB-5P-3400150P1, J7 CONNECTOR-HEADER-2X3P-3460180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, K3 BUTTON, K4 BUTTON, U1 CN3065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

Commit message: update design
Parts:
- added D14: SS54B, OPL:SMB
- added F2: 0.5A/15V, OPL_20130807:F1812
- added SJ17, SJ18, SJ19: JUMPER_2WLARGE, thewknd:JUMPER_LARGE_2WAY
- moved SJ15 5.12 mm to (98.4, 24.1)
- moved SJ10 5.02 mm to (84.8, 20.0), turned to 180 degrees
- moved R40 4.22 mm to (28.0, 43.5), turned to 270 degrees
- moved D3 2.36 mm to (19.2, 23.6), turned to 0 degrees
- moved C5 2.24 mm to (24.7, 20.8)
- moved D2 2.13 mm to (95.6, 25.4)
- moved SJ1 1.97 mm to (31.4, 23.4), turned to 270 degrees
- moved F1 1.80 mm to (28.8, 23.5)
- moved D7 1.59 mm to (96.7, 1.42)
- moved PAD6 0.32 mm to (88.9, 20.0)
- moved C7 0.20 mm to (21.6, 43.6)
- moved SJ7 0.20 mm to (21.6, 50.0)
- moved C2 0.10 mm to (15.2, 37.0)
- moved SJ12 0.10 mm to (15.2, 30.6)
Connections:
- new net N$59: D14.+, F2.2
- new net N$65: F2.1, SJ19.1
- net D6: now also SJ17.2
- net N$56: now also SJ17.1
- net VIN_T3_DIRECT: now also D14.-, SJ18.1
- net VUSB: now also SJ18.2, SJ19.2
Routing:
- net N$56: track 3.09 -> 30.2 mm
- net VUSB: track 104.1 -> 119.8 mm, vias 2 -> 3
- net N$59: track 0.00 -> 13.8 mm, vias 0 -> 2
- net VIN_T3_DIRECT: track 10.2 -> 23.8 mm
- net AREF: track 117.6 -> 125.0 mm, vias 7 -> 5
- net D6: track 57.4 -> 61.5 mm
- net N$65: track 0.00 -> 2.88 mm
- net VCC: track 58.4 -> 60.4 mm
- net N$34: track 1.59 -> 3.17 mm
- net 3.3V: track 355.4 -> 356.7 mm, vias 11 -> 12
- net N$36: track 51.7 -> 50.4 mm
- net ARDUINO_SHIELD_VIN_PIN: track 43.6 -> 44.9 mm
- net DIRECT_AREF: track 4.45 -> 5.63 mm
- net N$53: track 29.9 -> 29.2 mm
- net VBAT: track 93.8 -> 93.4 mm, vias 3 -> 5
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Other:
- board text added: "9.2013 L3.4.5"
- board text removed: "5.2013 L3.4.5"
