File: EAGLEPCB/board.sch (EAGLE design)
At the start: 125 parts, among them J1 JACK-DC-3P-3410020P1, J2 CONNECTOR-HEADER-10P-3460510P1, J3 CONNECTOR-HEADER-10P-3460510P1, J4 MICRO-SDCARD-CONNECTOR-330006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, J5 JST-2P-SMD-PW, J6 MICRO-USB-5P-3400150P1, J7 CONNECTOR-HEADER-2X3P-3460180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, K3 BUTTON, K4 BUTTON, Q1 MOSFET-P-0440210P1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

Commit message: update design
Parts:
- added D14: SS54B, OPL:D-SMB
- added F2: 0.5A/15V, OPL_20130807:FUSE-1812
- added SJ17, SJ18, SJ19: JUMPER_2WLARGE, thewknd:JUMPER_2WLARGE
Connections:
- new net N$59: D14.+, F2.2
- new net N$65: F2.1, SJ19.1
- net D6: now also SJ17.2
- net N$56: now also SJ17.1
- net VIN_T3_DIRECT: now also D14.-, SJ18.1
- net VUSB: now also SJ18.2, SJ19.2
Other:
- note added: "Battery"
- note added: "POWEREN#"
- moved on the sheet: R40
